Commit message: AIEAR: ros2_control migration (hardware interface + bringup)

File: src/aiear_robot/model/robot.xacro (robot description, xacro)
@@ -1,192 +1,230 @@
 <?xml version="1.0" encoding="UTF-8"?>
-<robot name="four_wheeled_diff_drive_robot" xmlns:xacro="http://www.ros.org/wiki/xacro">
-    <!-- Step 1: Defining Geometry and Constants -->
-    <!-- <xacro:property name="pi" value="3.14159265" /> -->
-    <!-- meters kgs and seconds are the SI units here -->
-    <!-- Body link Dimensions in meters-->
-    <xacro:property name="a" value="1.0" />
-    <xacro:property name="b" value="0.3" />
-    <xacro:property name="c" value="0.6" />
-    <!-- Wheel and Caster Dimensions for wheel 1 2 and caster -->
-    <!-- wheel and caster radius -->
-    <xacro:property name="r" value="0.15" />
-    <!-- wheel width (not diameter) -->
-    <xacro:property name="d" value="0.1" />
-    <xacro:property name="s1" value="${b/2+r}" />
-    <xacro:property name="s2" value="${2*r}" />
-    <xacro:property name="s3" value="${2*r}" />
-    <xacro:property name="s4" value="${c/2+d/2}" />
-    <!-- Define the Mass and inertia properties of the robot -->
-    <!-- densities for body link (box), wheel link(cylinder), and caster link (sphere) -->
-    <!-- body -->
-    <xacro:property name="d1" value="2710.0" />
-    <!-- wheel material density -->
-    <xacro:property name="d2" value="2710.0" />
-    <!-- Caster material density -->
-    <xacro:property name="d3" value="2710.0" />
-    <!-- robot body mass,wheelmass and caster mass -->
-    <!-- body -->
-    <xacro:property name="m1" value="${d1*a*b*c}" />
-    <!-- wheel -->
-    <xacro:property name="m2" value="${d2*pi*r*r*d}" />
-    <!-- caster -->
-    <xacro:property name="m3" value="${d3*(4.0/3.0)*pi*r*r*r}" />
-    <!-- Moments of intertia -->
-    <!-- of the robot body -->
-    <!-- x-axis -->
-    <xacro:property name="Ix_body" value="${(1.0/12.0)*m1*(b*b+c*c)}" />
-    <!-- y-axis-->
-    <xacro:property name="Iy_body" value="${(1.0/12.0)*m1*(a*a+b*b)}" />
-    <!-- z-axis -->
-    <xacro:property name="Iz_body" value="${(1.0/12.0)*m1*(a*a+c*c)}" />
-    <!-- of the wheel links -->
-    <!-- for x and y axis (same formula) -->
-    <xacro:property name="I_x_and_y_wheel" value="${(1.0/12.0)*m2*(3.0*r*r+d*d)}" />
-    <!-- for z axis -->
-    <xacro:property name="Iz" value="${0.5*m2*r*r}" />
-    <!-- of the caster sphere -->
-    <xacro:property name="I_x_and_y_and_z" value="${(2.0/5.0)*m3*r*r}" />
-    <!-- INERTIAL TAGS : defining the center of mass tags/frames -->
-    <xacro:macro name="inertia_body">
-        <inertial>
-            <!-- Displacement and orientation of center of mass frame of the link with repect to the fixed "world" -->
-            <origin rpy="0 0 0" xyz="0 0 ${s1}" />
-            <mass value="${m1}" />
-            <inertia ixx="${Ix_body}" ixy="0.0" ixz="0.0" iyy="${Iy_body}" iyz="0.0" izz="${Iz_body}" />
-        </inertial>
-    </xacro:macro>
-    <!-- This macro defines the complette inertial section of the wheel -->
-    <xacro:macro name="inertia_wheel">
-        <inertial>
-            <origin rpy="1.570795 0 0" xyz="0 0 0" />
-            <mass value="${m2}" />
-            <inertia ixx="${I_x_and_y_wheel}" ixy="0.0" ixz="0.0" iyy="${I_x_and_y_wheel}" iyz="0.0" izz="${Iz}" />
-        </inertial>
-    </xacro:macro>
-    <!-- The complete inertial section of the caster (whet forces are catingonn it by default)  -->
-    <xacro:macro name="inertia_caster">
-        <inertial>
-            <origin rpy="0 0 0" xyz="0 0 0" />
-            <mass value="${m3}" />
-            <inertia ixx="${I_x_and_y_and_z}" ixy="0.0" ixz="0.0" iyy="${I_x_and_y_and_z}" iyz="0.0" izz="${I_x_and_y_and_z}" />
-        </inertial>
-    </xacro:macro>
-    <!-- To be able to have gazebo functionalities and motion control driver, you need to import this cource file -->
+<robot name="aiear_robot" xmlns:xacro="http://www.ros.org/wiki/xacro">
+    <!-- ================================================================
+       ARGUMENTS & PROPERTIES
+       ================================================================ -->
+    <xacro:arg name="wheel_count" default="2" /> <!-- Supports 2 or 4 -->
+    <xacro:arg name="use_ros2_control" default="false" />
+    <xacro:arg name="is_sim" default="true" />
+    <!-- Chassis (Updated dimensions) -->
+    <xacro:property name="chassis_length" value="0.37" />
+    <xacro:property name="chassis_width" value="0.26" />
+    <xacro:property name="chassis_height" value="0.25" />
+    <xacro:property name="chassis_mass" value="3.0" />
+    <!-- Wheels (Updated dimensions) -->
+    <xacro:property name="wheel_radius" value="0.055" />
+    <xacro:property name="wheel_width" value="0.04" />
+    <xacro:property name="wheel_mass" value="0.3" />
+    <xacro:property name="wheelbase" value="0.24" />
+    <xacro:property name="wheel_y" value="${wheelbase/2.0}" />
+    <xacro:property name="wheel_z" value="${-chassis_height/2}" />
+    <!-- Wheel longitudinal positions -->
+    <xacro:property name="wheel_front_x" value="0.10" />
+    <xacro:property name="wheel_rear_x" value="-0.10" />
+    <!-- Caster (passive ball caster, ø50 mm) - Used in 2-wheel mode -->
+    <xacro:property name="caster_radius" value="0.040" />
+    <xacro:property name="caster_mass" value="0.05" />
+    <xacro:property name="caster_x" value="0.13" />
+    <xacro:property name="caster_z" value="${-(chassis_height/2 + wheel_radius - caster_radius)}" />
+    <!-- ================================================================
+       SENSORS (Based on AIEAR design)
+       ================================================================ -->
+    <!-- RPLiDAR A1 -->
+    <xacro:property name="lidar_radius" value="0.038" />
+    <xacro:property name="lidar_height" value="0.040" />
+    <xacro:property name="lidar_mass" value="0.17" />
+    <!-- Positioned at the TOP EDGE of the FRONT -->
+    <xacro:property name="lidar_x" value="${chassis_length/2 - lidar_radius}" />
+    <xacro:property name="lidar_z" value="${chassis_height/2 + lidar_height/2}" />
+    <!-- IMX500 Camera -->
+    <xacro:property name="cam_mass" value="0.05" />
+    <xacro:property name="cam_depth" value="0.025" />
+    <!-- Positioned at the FRONT FACE (middle) -->
+    <xacro:property name="cam_x" value="${chassis_length/2 + cam_depth/2}" />
+    <xacro:property name="cam_z" value="0" />
+    <xacro:property name="cam_pitch" value="0" /> <!-- Facing forward -->
+    <!-- ================================================================
+       INCLUDES
+       ================================================================ -->
     <xacro:include filename="$(find aiear_robot)/model/robot.gazebo" />
-    <!-- Defining the links and joints -->
-    <!-- Fictious link of the robot -->
-    <link name="base_footprint">
-        <!-- theres nothing in here ecause this is a fabricated link and is not part of the robot ...its more like a reference frame -->
-    </link>
-    <!-- Between every two links, there is a joint we need to define -->
-    <!-- in our case here the twolinks are the base_footprint(fictious link) and the body_link of the robot -->
-    <joint name="body_link_joint" type="fixed">
+    <!-- Optional: Include ROS2 Control if requested -->
+    <xacro:if value="$(arg use_ros2_control)">
+        <xacro:include filename="$(find aiear_robot)/model/ros2_control.xacro" />
+    </xacro:if>
+    <!-- ================================================================
+       INERTIA MACROS
+       ================================================================ -->
+    <xacro:macro name="box_inertia" params="m x y z">
+        <inertial>
+            <origin xyz="0 0 0" rpy="0 0 0" />
+            <mass value="${m}" />
+            <inertia ixx="${m*(y*y+z*z)/12}" ixy="0.0" ixz="0.0"
+                     iyy="${m*(x*x+z*z)/12}" iyz="0.0"
+                     izz="${m*(x*x+y*y)/12}" />
+        </inertial>
+    </xacro:macro>
+    <xacro:macro name="wheel_inertia" params="m r h">
+        <inertial>
+            <origin xyz="0 0 0" rpy="${pi/2} 0 0" />
+            <mass value="${m}" />
+            <inertia ixx="${m*(3*r*r+h*h)/12}" ixy="0.0" ixz="0.0"
+                     iyy="${m*r*r/2}" iyz="0.0"
+                     izz="${m*(3*r*r+h*h)/12}" />
+        </inertial>
+    </xacro:macro>
+    <xacro:macro name="cylinder_inertia_z" params="m r h">
+        <inertial>
+            <origin xyz="0 0 0" rpy="0 0 0" />
+            <mass value="${m}" />
+            <inertia ixx="${m*(3*r*r+h*h)/12}" ixy="0.0" ixz="0.0"
+                     iyy="${m*(3*r*r+h*h)/12}" iyz="0.0"
+                     izz="${m*r*r/2}" />
+        </inertial>
+    </xacro:macro>
+    <xacro:macro name="sphere_inertia" params="m r">
+        <inertial>
+            <origin xyz="0 0 0" rpy="0 0 0" />
+            <mass value="${m}" />
+            <inertia ixx="${2*m*r*r/5}" ixy="0.0" ixz="0.0"
+                     iyy="${2*m*r*r/5}" iyz="0.0"
+                     izz="${2*m*r*r/5}" />
+        </inertial>
+    </xacro:macro>
+    <!-- ================================================================
+       WHEEL MACRO
+       ================================================================ -->
+    <xacro:macro name="wheel" params="prefix x y">
+        <link name="${prefix}_wheel_link">
+            <visual>
+                <origin xyz="0 0 0" rpy="${pi/2} 0 0" />
+                <geometry>
+                    <cylinder radius="${wheel_radius}" length="${wheel_width}" />
+                </geometry>
+                <material name="black">
+                    <color rgba="0.1 0.1 0.1 1.0" />
+                </material>
+            </visual>
+            <collision>
+                <origin xyz="0 0 0" rpy="${pi/2} 0 0" />
+                <geometry>
+                    <cylinder radius="${wheel_radius}" length="${wheel_width}" />
+                </geometry>
+            </collision>
+            <xacro:wheel_inertia m="${wheel_mass}" r="${wheel_radius}" h="${wheel_width}" />
+        </link>
+        <joint name="${prefix}_wheel_joint" type="continuous">
+            <parent link="base_link" />
+            <child link="${prefix}_wheel_link" />
+            <origin xyz="${x} ${y} ${wheel_z}" rpy="0 0 0" />
+            <axis xyz="0 1 0" />
+            <dynamics damping="0.1" friction="0.1" />
+        </joint>
+    </xacro:macro>
+    <!-- ================================================================
+       LINKS & JOINTS
+       ================================================================ -->
+    <!-- base_footprint -->
+    <link name="base_footprint" />
+    <joint name="base_footprint_joint" type="fixed">
         <parent link="base_footprint" />
-        <child link="body_link" />
-    </joint>
-    <!-- ############################################## -->
-    <!-- START BODY LINK OF THE ROBOT -->
-    <!-- ############################################### -->
-    <link name="body_link">
+        <child link="base_link" />
+        <origin xyz="0 0 ${wheel_radius + chassis_height/2}" rpy="0 0 0" />
+    </joint>
+    <!-- base_link (Chassis) -->
+    <link name="base_link">
         <visual>
-            <!-- <origin xyz="0 0 0" rpy="0 0 ${s1}" /> -->
-            <origin xyz="0 0 0" rpy="0 0 0" />
-            <geometry>
-                <box size="${a} ${c} ${b}" />
-            </geometry>
+            <origin xyz="0 0 0" rpy="0 0 0" />
+            <geometry>
+                <box size="${chassis_length} ${chassis_width} ${chassis_height}" />
+            </geometry>
+            <material name="blue">
+                <color rgba="0.0 0.0 0.8 1.0" />
+            </material>
         </visual>
         <collision>
-            <!-- <origin xyz="0 0 0" rpy="0 0 ${s1}" /> -->
-            <origin xyz="0 0 0" rpy="0 0 0" />
-            <geometry>
-                <box size="${a} ${c} ${b}" />
+            <origin xyz="0 0 0" rpy="0 0 0" />
+            <geometry>
+                <box size="${chassis_length} ${chassis_width} ${chassis_height}" />
             </geometry>
         </collision>
-        <xacro:inertia_body />
+        <xacro:box_inertia m="${chassis_mass}" x="${chassis_length}" y="${chassis_width}" z="${chassis_height}" />
     </link>
-    <!-- ############################################## -->
-    <!-- END BODY LINK OF THE ROBOT -->
-    <!-- ############################################### -->
-    <!-- ############################################## -->
-    <!-- START Wheel links of Robot and their joints -->
-    <!-- ############################################### -->
-    <!-- Joint btn wheel 1 and body link -->
-    <joint name="wheel1_joint" type="continuous">
-        <parent link="body_link" />
-        <child link="wheel1_link" />
-        <!-- <origin xyz="${-s2} ${-s4} ${r}" rpy="0 0 0" /> -->
-        <origin xyz="0 0 0" rpy="1.570796327 0 0" />
-        <axis xyz="0 1 0" />  <!-- This one determins in which axis is your link performing the motion -->
-        <limit effort="50000" velocity="10" /> <!-- Effort = max Torque vel = max vel -->
-        <dynamics damping="1.0" friction="1.0"/>
-    </joint>
-    <!-- Wheel 1 link -->
-    <link name="wheel1_link">
+    <!-- Wheel Configuration Logic -->
+    <xacro:if value="${'$(arg wheel_count)' == '2'}">
+        <!-- 2-Wheel Mode: Middle drive wheels + Front Caster -->
+        <xacro:wheel prefix="left" x="0" y="${wheel_y}" />
+        <xacro:wheel prefix="right" x="0" y="${-wheel_y}" />
+        <!-- Caster -->
+        <link name="caster_link">
+            <visual>
+                <geometry>
+                    <sphere radius="${caster_radius}" />
+                </geometry>
+                <material name="grey">
+                    <color rgba="0.5 0.5 0.5 1.0" />
+                </material>
+            </visual>
+            <collision>
+                <geometry>
+                    <sphere radius="${caster_radius}" />
+                </geometry>
+            </collision>
+            <xacro:sphere_inertia m="${caster_mass}" r="${caster_radius}" />
+        </link>
+        <joint name="caster_joint" type="fixed">
+            <parent link="base_link" />
+            <child link="caster_link" />
+            <origin xyz="${caster_x} 0 ${caster_z}" rpy="0 0 0" />
+        </joint>
+    </xacro:if>
+    <xacro:if value="${'$(arg wheel_count)' == '4'}">
+        <!-- 4-Wheel Mode: Front and Rear drive wheels -->
+        <xacro:wheel prefix="front_left" x="${wheel_front_x}" y="${wheel_y}" />
+        <xacro:wheel prefix="front_right" x="${wheel_front_x}" y="${-wheel_y}" />
+        <xacro:wheel prefix="rear_left" x="${wheel_rear_x}" y="${wheel_y}" />
+        <xacro:wheel prefix="rear_right" x="${wheel_rear_x}" y="${-wheel_y}" />
+    </xacro:if>
+    <!-- LiDAR -->
+    <link name="lidar_link">
         <visual>
-            <!-- <origin xyz="1.570795 0 0" rpy="0 0 0" /> -->
-            <origin xyz="0 0 0" rpy="0 0 0" />
-            <geometry>
-                <cylinder radius="${d}" length="${r}" />
-            </geometry>
+            <geometry>
+                <cylinder radius="${lidar_radius}" length="${lidar_height}" />
+            </geometry>
+            <material name="dark_grey"><color rgba="0.2 0.2 0.2 1.0" /></material>
         </visual>
         <collision>
-            <!-- <origin xyz="1.570795 0 0" rpy="0 0 0" /> -->
-             <origin xyz="0 0 0" rpy="0 0 0" />
-            <geometry>
-                <cylinder radius="${d}" length="${r}" />
+            <geometry>
+                <cylinder radius="${lidar_radius}" length="${lidar_height}" />
             </geometry>
         </collision>
-        <xacro:inertia_wheel />
+        <xacro:cylinder_inertia_z m="${lidar_mass}" r="${lidar_radius}" h="${lidar_height}" />
     </link>
-    <!-- Joint btn wheel 2 and body link -->
-     <joint name="wheel2_joint" type="continuous">
-        <parent link="body_link" />
-        <child link="wheel2_link" />
-        <origin xyz="${s2} ${s4} ${r}" rpy="0 0 0" />
-        <axis xyz="0 1 0" />
-        <limit  effort="50000" velocity="10" />
-        <dynamic damping="1.0" friction="1.0" />
-     </joint>
-    <!-- Wheel 2 link -->
-     <link name="wheel2_link">
+    <joint name="lidar_joint" type="fixed">
+        <parent link="base_link" />
+        <child link="lidar_link" />
+        <origin xyz="${lidar_x} 0 ${lidar_z}" rpy="0 0 0" />
+    </joint>
+    <!-- Camera -->
+    <link name="camera_link">
         <visual>
-            <origin xyz="1.570795 0 0" rpy="0 0 0" />
-            <geometry>
-                <cylinder radius="${d}" length="${r}" />
-            </geometry>
+            <geometry><box size="0.025 0.090 0.025" /></geometry>
+            <material name="black" />
         </visual>
         <collision>
-            <origin xyz="1.570795 0 0" rpy="0 0 0" />
-            <geometry>
-                <cylinder radius="${d}" length="${r}" />
-            </geometry>
+            <geometry><box size="0.025 0.090 0.025" /></geometry>
         </collision>
-        <xacro:inertia_wheel />
-     </link>
-    <!-- ############################################## -->
-    <!-- End Wheel links of Robot and their joints -->
-    <!-- ############################################### -->
-    <!-- ############################################## -->
-    <!-- START Caster link of Robot and joint -->
-    <!-- ############################################### -->
-    <joint name="caster_joint" type="fixed">
-        <parent link="body_link" />
-        <child link="caster_link" />
-        <origin xyz="${s3} 0 ${r}" rpy="0 0 0" />
-    </joint>
-    <link name="caster_link">
-        <visual>
-            <origin xyz="0 0 0" rpy="0 0 0" />
-            <geometry>
-                <sphere radius="${r}" />
-            </geometry>
-        </visual>
-        <collision>
-            <origin xyz="0 0 0" rpy="0 0 0" />
-            <geometry>
-                <sphere radius="${r}" />
-            </geometry>
-        </collision>
-        <xacro:inertia_caster />
+        <xacro:box_inertia m="${cam_mass}" x="0.025" y="0.090" z="0.025" />
     </link>
+    <joint name="camera_joint" type="fixed">
+        <parent link="base_link" />
+        <child link="camera_link" />
+        <origin xyz="${cam_x} 0 ${cam_z}" rpy="0 ${cam_pitch} 0" />
+    </joint>
+    <!-- Camera optical frame -->
+    <link name="camera_optical_link" />
+    <joint name="camera_optical_joint" type="fixed">
+        <parent link="camera_link" />
+        <child link="camera_optical_link" />
+        <origin xyz="0 0 0" rpy="${-pi/2} 0 ${-pi/2}" />
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