Commit message: Tune skid-steer: wheel_separation 1.373, angular cap 0.8, SLAM thresholds 0.1

File: src/aiear_robot/model/ros2_control.xacro (robot description, xacro)
@@ -10,5 +10,5 @@
                 <!-- This is where the real hardware plugin goes in the future -->
                 <plugin>aiear_hardware/AiearSystemHardware</plugin>
-                <param name="serial_port">/dev/ttyUSB0</param>
+                <param name="serial_port">/dev/aiear_esp32</param>
             </xacro:unless>
         </hardware>

File: src/aiear_robot/urdf/aiear.urdf.xacro (robot description, xacro)
@@ -80,8 +80,7 @@
   </link>
   <joint name="laser_joint" type="fixed">
-    <parent link="base_link" />
-    <child link="laser" />
-    <!-- z: height above chassis bottom, converted to base_link-center frame -->
-    <origin xyz="${lidar_x} 0 ${lidar_height - body_height/2}" rpy="0 0 0" />
+    <parent link="base_link"/>
+    <child link="laser"/>
+    <origin xyz="0.163 0 ${0.32 - body_height/2}" rpy="0 0 3.14159"/>
   </joint>
   <!-- ======================= ros2_control =========================== -->
